File: pcb/reworkctf.sch (KiCad schematic (older format))
At the start: 41 parts

Commit message: Finished initial work on reworkctf schematic and documentation
Parts:
- added C1, C2, C25, C26, C27, C29, C3, C4: 4.7 uF, symbol C
- added C10, C11, C12, C13, C14, C15, C16, C17, C18, C19, C28, C30, C31, C32, C33, C34, C35, C36, C37, C38, C39, C5, C6, C7, C8, C9: 0.1 uF, symbol C
- added D17, D18, D19, D20, D21, D22, D23: GREEN, symbol LED
- added R1, R10, R2, R28, R29, R3, R4, R5, R6, R7, R8, R9: 1K, symbol R
- added R27, R46, R47, R48, R49, R50, R51: 470, symbol R
- added R30, R41, R42, R44, R45: 0, symbol R
- added R31, R32, R33, R34, R35, R36, R37, R38, R39, R40, R43: 270, symbol R
- added U2: W25Q80BV, symbol W25Q80BV
- added U3, U6: 74HC04, symbol 7404_BLOCK
- added U4: OSC, symbol OSC
- added W1, W2, W3, W4, W5, W6: VIAPAD, symbol TEST_1P
- gave numbers to parts that had none: 41
Connections:
- net 1V2: now also C25.1, C27.1, C29.1, C31.1, C33.1, C35.1, C36.1, C37.1, C38.1
- net 2V5: now also J1.2 (Vccaux), U1.B13 (VCCO0), U1.B5 (VCCO0), U1.B9 (VCCO0), U1.E8 (VCCO0), C26.1, C28.1, C30.1, C32.1, C34.1, R1.1, R2.2
- net 3V3: now also U1.D2 (VCCO3), U1.E15 (VCCO1), U1.H12 (VCCO1), U1.H2 (VCCO3), U1.J15 (VCCO1), U1.J5 (VCCO3), U1.M2 (VCCO3), U1.M9 (VCCO2), U1.N14 (IO_L01N_1/LDC2), U1.N15 (VCCO1), U1.R12 (VCCO2), U1.R4 (VCCO2), U1.R8 (VCCO2), C1.1, C10.1, C11.1, C12.1, C13.1, C14.1, C15.1, C16.1, C17.2, C18.2, C19.2, C2.1, C3.1, C39.2, C4.1, C5.1, C6.1, C7.1, C8.1, C9.1, R10.1, R28.2, R29.1, R4.1, R5.1, R6.1, R7.1, U2.8 (VCC), U3.14 (VDD), U4.1 (E/D#), U4.4 (Vdd), U6.14 (VDD)
- net GND: now also U1.A1 (GND), U1.A16 (GND), U1.B11 (GND), U1.B7 (GND), U1.C14 (GND), U1.C3 (GND), U1.E12 (GND), U1.E5 (GND), U1.F2 (GND), U1.F6 (GND), U1.G10 (GND), U1.G15 (GND), U1.G8 (GND), U1.H9 (GND), U1.J8 (GND), U1.K2 (GND), U1.K7 (GND), U1.K9 (GND), U1.L11 (GND), U1.L15 (GND), U1.M12 (GND), U1.M5 (GND), U1.N8 (IO_L08N_2/D4), U1.P14 (GND), U1.P3 (GND), U1.R10 (GND), U1.R6 (GND), U1.T1 (GND), U1.T16 (GND), C1.2, C10.2, C11.2, C12.2, C13.2, C14.2, C15.2, C16.2, C17.1, C18.1, C19.1, C2.2, C25.2, C26.2, C27.2, C28.2, C29.2, C3.2, C30.2, C31.2, C32.2, C33.2, C34.2, C35.2, C36.2, C37.2, C38.2, C39.1, C4.2, C5.2, C6.2, C7.2, C8.2, C9.2, D17.1 (K), D18.1 (K), D19.1 (K), D20.1 (K), D21.1 (K), D22.1 (K), D23.1 (K), R3.2, R43.1, R8.1, R9.1, U2.4 (GND), U3.7 (VSS), U4.2 (Vss), U6.13 (6A), U6.7 (VSS)
- net LEVEL10_OK: now also U1.K1 (IO_L15N_3/LHCLK7)
- net LEVEL11_OK: now also U1.J2 (IO_L14P_3/LHCLK4)
- net LEVEL12_OK: now also U1.J1 (IO_L14N_3/LHCLK5)
- net LEVEL13_OK: now also U1.H3 (IO_L12P_3/LHCLK2)
- net LEVEL14_OK: now also U1.J3 (IO_L12N_3/IRDY2/LHCLK3)
- net LEVEL15_OK: now also U1.G2 (IO_L11P_3/LHCLK0)
- net LEVEL16_OK: now also U1.H1 (IO_L11N_3/LHCLK1)
- net LEVEL1_OK: now also U1.N3 (IO_L24P_3)
- net LEVEL2_OK: now also U1.M4 (IO_L24N_3)
- net LEVEL3_OK: now also U1.R1 (IO_L23P_3)
- net LEVEL4_OK: now also U1.P2 (IO_L23N_3)
- net LEVEL5_OK: now also U1.N2 (IO_L22P_3)
- net LEVEL6_OK: now also U1.P1 (IO_L22N_3)
- net LEVEL7_OK: now also U1.M1 (IO_L20P_3)
- net LEVEL8_OK: now also U1.N1 (IO_L20N_3)
- net LEVEL9_OK: now also U1.K3 (IO_L15P_3/TRDY2/LHCLK6)
- net LEVEL15_TEST_N: now reaches U1.A11 (IO_L07N_0)
- net LEVEL15_TEST_N: now also U1.C10 (IO_L09P_0/GCLK4)
- net FPGA_RST_N: now reaches U1.A2 (/PROG)
- net FPGA_RST_N: now also R1.2
- net LEVEL22_OK: now reaches U1.C1 (IO_L01N_3)
- net LEVEL22_OK: now also R51.2
- net LEVEL15_TEST_P: now reaches U1.C11 (IO_L07P_0)
- net LEVEL15_TEST_P: now also U1.D9 (IO_L09N_0/GCLK5)
- net LEVEL7_TEST_N: now reaches U1.C12 (IO_L03P_0)
- net LEVEL7_TEST_N: now also U1.C13 (IO_L01N_0)
- net LEVEL21_OK: now reaches U1.C2 (IO_L01P_3)
- net LEVEL21_OK: now also R50.2
- net LEVEL17_OK: now reaches U1.D1 (IO_L03P_3)
- net LEVEL17_OK: now also R46.2
- net LEVEL7_TEST_P: now reaches U1.D11 (IO_L03N_0)
- net LEVEL7_TEST_P: now also U1.D13 (IO_L01P_0)
- net LEVEL20_OK: now reaches U1.D3 (IO_L02N_3)
- net LEVEL20_OK: now also R49.2
- net LEVEL19_OK: now reaches U1.D4 (IO_L02P_3)
- net LEVEL19_OK: now also R48.2
- net at U1.D5 (IO_L20N_0/PUDC_B): now also R2.1
- net LEVEL18_OK: now reaches U1.E1 (IO_L03N_3)
- net LEVEL18_OK: now also R47.2
- net LEVEL11_TEST: now reaches U1.E2 (IO_L05N_3_NC_IN_50A)
- net LEVEL11_TEST: now also R45.2
- net LEVEL11_SENSE: now reaches U1.E3 (IO_L05P_3_NC_IN_50A)
- net LEVEL11_SENSE: now also U6.6 (3Y)
- net LEVEL9_SENSE: now reaches U1.E4 (IP_L04P_3)
- net LEVEL9_SENSE: now also R40.1
- net at U1.F1 (IO_L08P_3): now also R39.2
- net LEVEL9_TEST: now reaches U1.F3 (IO_L07P_3_NC_IN_50A)
- net LEVEL9_TEST: now also R40.2
- net LEVEL10_SENSE: now reaches U1.F4 (IP_L04N_3/VREF_3)
- net LEVEL10_SENSE: now also U6.4 (2Y)
- net LEVEL8_TEST: now reaches U1.G1 (IO_L08N_3/VREF_3)
- net LEVEL8_TEST: now also U6.1 (1A)
- net at U1.G3 (IO_L09P_3_NC_IN_50A): now also R30.2
- net LEVEL10_TEST: now reaches U1.G4 (IO_L07N_3_NC_IN_50A)
- net LEVEL10_TEST: now also R44.2
- net at U1.H4 (IO_L09N_3_NC_IN_50A): now also R38.2
- net LEVEL3_TEST: now reaches U1.H5 (IO_L10N_3_NC_IN_50A)
- net LEVEL3_TEST: now also U3.11 (5A)
- net at U1.H6 (IO_L10P_3_NC_IN_50A): now also R31.2
- net LEVEL6_SENSE: now reaches U1.H7 (IP_L13P_3)
- net LEVEL6_SENSE: now also U3.6 (3Y)
- net LEVEL18_SENSE: now reaches U1.J12 (IO_L10P_1/A8)
- net LEVEL18_SENSE: now also W1.1
- net LEVEL18_TEST: now reaches U1.J13 (IO_L10N_1/A9)
- net LEVEL18_TEST: now also W3.1
- net LEVEL22_TEST: now reaches U1.J16 (IO_L12N_1/TRDY1/RHCLK3)
- net LEVEL22_TEST: now also W4.1
- net LEVEL8_SENSE: now reaches U1.J7 (IP_L13N_3)
- net LEVEL8_SENSE: now also U6.2 (1Y)
- net at U1.K14 (IO_L11N_1/RHCLK1): now also R35.1
- net LEVEL21_SENSE: now reaches U1.K15 (IO_L11P_1/RHCLK0)
- net LEVEL21_SENSE: now also U6.10 (5Y)
- net LEVEL22_SENSE: now reaches U1.K16 (IO_L12P_1/RHCLK2)
- net LEVEL22_SENSE: now also W2.1
- net LEVEL4_SENSE: now reaches U1.K5 (IP_L21P_3)
- net LEVEL4_SENSE: now also U3.8 (4Y)
- net LEVEL5_SENSE: now reaches U1.K6 (IP_L21N_3)
- net LEVEL5_SENSE: now also U3.4 (2Y)
- net LEVEL14_SENSE: now reaches U1.L10 (IP_2/VREF_2)
- net LEVEL14_SENSE: now also U6.8 (4Y)
- net LEVEL1_SENSE: now reaches U1.L5 (IP_L25P_3)
- net LEVEL1_SENSE: now also U3.12 (6Y)
- net LEVEL3_SENSE: now reaches U1.L6 (IP_L25N_3/VREF_3)
- net LEVEL3_SENSE: now also U3.10 (5Y)
- net LEVEL12_SENSE: now reaches U1.L7 (IP_2)
- net LEVEL12_SENSE: now also U3.2 (1Y)
- net LEVEL13_TEST_B: now reaches U1.L8 (IP_2)
- net LEVEL13_TEST_B: now also R37.1
- net LEVEL13_TEST_A: now reaches U1.L9 (IP_2/VREF_2)
- net LEVEL13_TEST_A: now also R36.1
- net LEVEL16_TEST_C: now reaches U1.M13 (IO_L05P_1_NC_IN_50A)
- net LEVEL16_TEST_C: now also R34.2
- net LEVEL16_TEST_B: now reaches U1.M14 (IO_L05N_1/VREF_1_NC_IN_50A)
- net LEVEL16_TEST_B: now also R33.2
- net at U1.N11 (IO_L16N_2): now also R37.2
- net at U1.N13 (IO_L01P_1/HDC): now also R32.1
- net at U1.N4 (IO_L01P_2/M1): now also R9.2
- net at U1.N6 (IO_L04P_2/VS1): now also R5.2
- net CLK_1MHZ: now reaches U1.N9 (IO_L11P_2/GCLK0)
- net CLK_1MHZ: now also U4.3 (CLK)
- net SPI_MOSI: now reaches U1.P10 (IO_L14N_2/MOSI/CSI_B)
- net SPI_MOSI: now also U2.5 (DI/IO0)
- net at U1.P11 (IO_L16P_2): now also R36.2
- net at U1.P15 (IO_L02N_1/LDC0): now also R33.1
- net LEVEL16_TEST_A: now reaches U1.P16 (IO_L03P_1/A0)
- net LEVEL16_TEST_A: now also R32.2
- net at U1.P4 (IO_L01N_2/M0): now also R10.2
- net at U1.P5 (IO_L04N_2/VS0): now also R6.2
- net LEVEL17_TEST: now reaches U1.P7 (IO_L08P_2/D5)
- net LEVEL17_TEST: now also R43.2
- net LEVEL19_SENSE: now reaches U1.P8 (IO_L10P_2/GCLK14)
- net LEVEL19_SENSE: now also U1.T5 (IO_L06P_2/D7), R41.1, R42.1
- net LEVEL14_TEST: now reaches U1.R11 (IO_L15N_2/DOUT)
- net LEVEL14_TEST: now also U6.8 (4Y)
- net SPI_SCK: now reaches U1.R14 (IO_L20N_2/CCLK)
- net SPI_SCK: now also U2.6 (CLK)
- net at U1.R15 (IO_L02P_1/LDC1): now also R34.1
- net at U1.R16 (SUSPEND): now also R3.1
- net at U1.R2 (IO_L02P_2/M2): now also R8.2
- net at U1.T12 (IO_L17P_2/INIT_B): now also R4.2
- net LEVEL12_TEST: now reaches U1.T13 (IO_L18P_2/D2)
- net LEVEL12_TEST: now also W5.1
- net SPI_MISO: now reaches U1.T14 (IO_L20P_2/D0/DIN/MISO)
- net SPI_MISO: now also U2.2 (DO/IO1)
- net FPGA_DONE: now reaches U1.T15 (DONE)
- net FPGA_DONE: now also R27.2
- net SPI_CS_N: now reaches U1.T2 (IO_L02N_2/CSO_B)
- net SPI_CS_N: now also U2.1 (CS#)
- net at U1.T3 (IO_L03N_2/VS2): now also R7.2
- net LEVEL19_TEST: now reaches U1.T6 (IO_L06N_2/D6)
- net LEVEL19_TEST: now also U1.T8 (IO_L10N_2/GCLK15), R41.2, R42.2
- new net: D17.2 (A), R27.1
- new net: R28.1, U2.3 (WP#/IO2)
- new net: R29.2, U2.7 (HOLD#/IO3)
- new net: R44.1, U6.3 (2A)
- new net: R45.1, U6.5 (3A)
- new net: D18.2 (A), R46.1
- new net: D19.2 (A), R47.1
- new net: D20.2 (A), R48.1
- new net: D21.2 (A), R49.1
- new net: D22.2 (A), R50.1
- new net: D23.2 (A), R51.1
- new net LEVEL12_TEST_FLOAT: U3.1 (1A), W6.1
- new net LEVEL1_TEST: R31.1, U3.13 (6A)
- new net LEVEL21_TEST: R35.2, U6.11 (5A)
- new net LEVEL4_TEST: R30.1, U3.8 (4Y)
- new net LEVEL5_TEST: R38.1, U3.3 (2A)
- new net LEVEL6_TEST: R39.1, U3.5 (3A)
- no-connect marks 48 -> 121
Other:
- note added: "FPGA decoupling"
- note added: "IO_L03 pair\nintentionally swapped"
- note added: "IO_L09 pair\nintentionally swapped"
- note added: "This via is level 20"
- note removed: "LEDs run from 3V3\nAt 2.2V typ Vf, 470R -> 2.3 mA"

Commit message: Initial work on layout
Parts:
- added C40, C41: 4.7 uF, azonenberg_pcb:EIA_0603_CAP_NOSILK, symbol C
- added C? (x4): 0.1 uF, azonenberg_pcb:EIA_0402_CAP_NOSILK, symbol C
- C1, C2, C20, C21, C22, C23, C24, C25, C26, C27, C29, C3, C4: footprint (none) -> azonenberg_pcb:EIA_0603_CAP_NOSILK
- C10, C11, C12, C13, C14, C15, C16, C17, C18, C19, C28, C30, C31, C32, C33, C34, C35, C36, C37, C38, C39, C5, C6, C7, C8, C9: footprint (none) -> azonenberg_pcb:EIA_0402_CAP_NOSILK
- D1, D10, D11, D12, D13, D14, D15, D16, D17, D18, D19, D2, D20, D21, D22, D23, D3, D4, D5, D6, D7, D8, D9: footprint (none) -> azonenberg_pcb:EIA_0603_LED
- J1: footprint (none) -> azonenberg_pcb:XILINX_JTAG_PTH_MOLEX_0878311420
- J2: footprint (none) -> azonenberg_pcb:CONN_HIROSE_UX60S-MB-5ST_MINI_USB
- R1, R10, R11, R12, R13, R14, R15, R16, R17, R18, R19, R2, R20, R21, R22, R23, R24, R25, R26, R27, R28, R29, R3, R31, R32, R33, R34, R35, R36, R37, R38, R39, R4, R41, R42, R43, R44, R46, R47, R48, R49, R5, R50, R51, R6, R7, R8, R9: footprint (none) -> azonenberg_pcb:EIA_0402_RES_NOSILK
- R30: footprint (none) -> azonenberg_pcb:EIA_0805_CAP_NOSILK
- R40: footprint (none) -> azonenberg_pcb:EIA_01005_RES_NOSILK
- R45: footprint (none) -> azonenberg_pcb:EIA_0201_RES_NOSILK
- U1: footprint (none) -> azonenberg_pcb:BGA_256_17x17_FULLARRAY_1MM
- U2: footprint (none) -> azonenberg_pcb:SOIC_8_3.9MM
- U3: footprint (none) -> azonenberg_pcb:SOIC_14_3.9MM_NOPIN11
- U4: value OSC -> 1 MHz; footprint (none) -> azonenberg_pcb:OSCILLATOR_3.2x2.5
- U5: footprint (none) -> azonenberg_pcb:QFN_16_0.5MM_3x3MM
- U6: footprint (none) -> azonenberg_pcb:TSSOP_14_0.65MM_5p6MM_NOPINS_1_2
- W1, W2, W3, W4, W5, W6: footprint (none) -> azonenberg_pcb:TESTPOINT_SMT_0.5MM
Connections:
- net 2V5: now also C?.1, C?.1, C?.1, C?.1
- net 5V0: now also C40.1, C41.1
- net GND: now also C40.2, C41.2, C?.2, C?.2, C?.2, C?.2

Commit message: Continued initial layout
Parts:
- added R?: 1K, azonenberg_pcb:EIA_0402_RES_NOSILK, symbol R
- gave numbers to parts that had none: 4
Connections:
- net 3V3: now also R?.2
- net SPI_CS_N: now also R?.1
Changed lines of the file:
@@
 5V0
 $Comp
-L C C?
+L C C42
 U 1 1 592BCB20
 P 3200 15200
-F 0 "C?" H 3315 15246 50  0000 L CNN
+F 0 "C42" H 3315 15246 50  0000 L CNN
 F 1 "0.1 uF" H 3315 15155 50  0000 L CNN
 F 2 "azonenberg_pcb:EIA_0402_CAP_NOSILK" H 3238 15050 50  0001 C CNN
@@
 $EndComp
 $Comp
-L C C?
+L C C43
 U 1 1 592BCC4C
 P 3700 15200
-F 0 "C?" H 3815 15246 50  0000 L CNN
+F 0 "C43" H 3815 15246 50  0000 L CNN
 F 1 "0.1 uF" H 3815 15155 50  0000 L CNN
 F 2 "azonenberg_pcb:EIA_0402_CAP_NOSILK" H 3738 15050 50  0001 C CNN
@@
 $EndComp
 $Comp
-L C C?
+L C C44
 U 1 1 592BCD7E
 P 4200 15200
-F 0 "C?" H 4315 15246 50  0000 L CNN
+F 0 "C44" H 4315 15246 50  0000 L CNN
 F 1 "0.1 uF" H 4315 15155 50  0000 L CNN
 F 2 "azonenberg_pcb:EIA_0402_CAP_NOSILK" H 4238 15050 50  0001 C CNN
@@
 $EndComp
 $Comp
-L C C?
+L C C45
 U 1 1 592BCEAE
 P 4700 15200
-F 0 "C?" H 4815 15246 50  0000 L CNN
+F 0 "C45" H 4815 15246 50  0000 L CNN
 F 1 "0.1 uF" H 4815 15155 50  0000 L CNN
 F 2 "azonenberg_pcb:EIA_0402_CAP_NOSILK" H 4738 15050 50  0001 C CNN
@@
 Connection ~ 3700 15050
 Connection ~ 4200 15050
+$Comp
+L R R?
+U 1 1 592C256B
+P 8800 1350
+F 0 "R?" V 8750 1200 50  0000 C CNN
+F 1 "1K" V 8800 1350 50  0000 C CNN
+F 2 "azonenberg_pcb:EIA_0402_RES_NOSILK" V 8730 1350 50  0001 C CNN
+F 3 "" H 8800 1350 50  0000 C CNN
+	1    8800 1350
+	-1   0    0    1
+$EndComp
+Text Label 8650 1200 2    60   ~ 0
+3V3
+Wire Wire Line
+	8650 1200 8800 1200
 $EndSCHEMATC

Commit message: Continued work on initial layout
Parts:
- gave numbers to parts that had none: 1
Connections:
- net LEVEL10_OK: now also U1.J1 (IO_L14N_3/LHCLK5); no longer U1.K1 (IO_L15N_3/LHCLK7)
- net LEVEL12_OK: now also U1.K1 (IO_L15N_3/LHCLK7); no longer U1.J1 (IO_L14N_3/LHCLK5)
- net LEVEL13_OK: now also U1.K3 (IO_L15P_3/TRDY2/LHCLK6); no longer U1.H3 (IO_L12P_3/LHCLK2)
- net LEVEL14_OK: now also U1.M1 (IO_L20P_3); no longer U1.J3 (IO_L12N_3/IRDY2/LHCLK3)
- net LEVEL15_OK: now also U1.N1 (IO_L20N_3); no longer U1.G2 (IO_L11P_3/LHCLK0)
- net LEVEL16_OK: now also U1.N2 (IO_L22P_3); no longer U1.H1 (IO_L11N_3/LHCLK1)
- net LEVEL17_OK: now also U1.P1 (IO_L22N_3); no longer U1.D1 (IO_L03P_3)
- net LEVEL18_OK: now also U1.P2 (IO_L23N_3); no longer U1.E1 (IO_L03N_3)
- net LEVEL19_OK: now also U1.R1 (IO_L23P_3); no longer U1.D4 (IO_L02P_3)
- net LEVEL1_OK: now also U1.C1 (IO_L01N_3); no longer U1.N3 (IO_L24P_3)
- net LEVEL20_OK: now also U1.M4 (IO_L24N_3); no longer U1.D3 (IO_L02N_3)
- net LEVEL22_OK: now also U1.N3 (IO_L24P_3); no longer U1.C1 (IO_L01N_3)
- net LEVEL2_OK: now also U1.D1 (IO_L03P_3); no longer U1.M4 (IO_L24N_3)
- net LEVEL3_OK: now also U1.D3 (IO_L02N_3); no longer U1.R1 (IO_L23P_3)
- net LEVEL3_TEST: now also U1.T9 (IO_L12N_2/GCLK3); no longer U1.H5 (IO_L10N_3_NC_IN_50A)
- net LEVEL4_OK: now also U1.E1 (IO_L03N_3); no longer U1.P2 (IO_L23N_3)
- net LEVEL5_OK: now also U1.F1 (IO_L08P_3); no longer U1.N2 (IO_L22P_3)
- net LEVEL6_OK: now also U1.F3 (IO_L07P_3_NC_IN_50A); no longer U1.P1 (IO_L22N_3)
- net LEVEL7_OK: now also U1.G1 (IO_L08N_3/VREF_3); no longer U1.M1 (IO_L20P_3)
- net LEVEL8_OK: now also U1.H1 (IO_L11N_3/LHCLK1); no longer U1.N1 (IO_L20N_3)
- net LEVEL8_TEST: now also U1.G2 (IO_L11P_3/LHCLK0); no longer U1.G1 (IO_L08N_3/VREF_3)
- net LEVEL9_OK: now also U1.H3 (IO_L12P_3/LHCLK2); no longer U1.K3 (IO_L15P_3/TRDY2/LHCLK6)
- net LEVEL9_TEST: now also U1.D4 (IO_L02P_3); no longer U1.F3 (IO_L07P_3_NC_IN_50A)
- net at R39.2: now also U1.T10 (IO_L14P_2); no longer U1.F1 (IO_L08P_3)
- net at U1.G3 (IO_L09P_3_NC_IN_50A): no longer R30.2
- net at U1.H4 (IO_L09N_3_NC_IN_50A): no longer R38.2
- net at U1.H6 (IO_L10P_3_NC_IN_50A): no longer R31.2
- net at U1.R5 (IO_L05N_2): now also R38.2
- net at U1.R9 (IO_L12P_2/GCLK2): now also R31.2
- net at U1.T4 (IO_L05P_2): now also R30.2
Other:
- moved on the sheet: R30, R31, R38, R39, R40
Changed lines of the file:
@@
 NoConn ~ 7000 4750
 NoConn ~ 7000 4850
-NoConn ~ 7000 4950
-NoConn ~ 7000 5050
 NoConn ~ 2700 3650
 NoConn ~ 2700 3850
@@
 	0    1    1    0
 $EndComp
-Text Label 7200 3550 0    60   ~ 0
+Text Label 7200 7450 0    60   ~ 0
 LEVEL1_OK
-Text Label 7200 3650 0    60   ~ 0
+Text Label 7200 6950 0    60   ~ 0
 LEVEL2_OK
-Text Label 7200 3750 0    60   ~ 0
+Text Label 7200 7250 0    60   ~ 0
 LEVEL3_OK
-Text Label 7200 3850 0    60   ~ 0
+Text Label 7200 7050 0    60   ~ 0
 LEVEL4_OK
-Text Label 7200 3950 0    60   ~ 0
+Text Label 7200 6350 0    60   ~ 0
 LEVEL5_OK
-Text Label 7200 4050 0    60   ~ 0
+Text Label 7200 6550 0    60   ~ 0
 LEVEL6_OK
-Text Label 7200 4150 0    60   ~ 0
+Text Label 7200 6450 0    60   ~ 0
 LEVEL7_OK
-Text Label 7200 4250 0    60   ~ 0
+Text Label 7200 5850 0    60   ~ 0
 LEVEL8_OK
-Text Label 7200 5150 0    60   ~ 0
+Text Label 7200 5550 0    60   ~ 0
 LEVEL9_OK
-Text Label 7200 5250 0    60   ~ 0
+Text Label 7200 5450 0    60   ~ 0
 LEVEL10_OK
 Text Label 7200 5350 0    60   ~ 0
 LEVEL11_OK
-Text Label 7200 5450 0    60   ~ 0
+Text Label 7200 5250 0    60   ~ 0
 LEVEL12_OK
-Text Label 7200 5550 0    60   ~ 0
+Text Label 7200 5150 0    60   ~ 0
 LEVEL13_OK
-Text Label 7200 5650 0    60   ~ 0
+Text Label 7200 4150 0    60   ~ 0
 LEVEL14_OK
-Text Label 7200 5750 0    60   ~ 0
+Text Label 7200 4250 0    60   ~ 0
 LEVEL15_OK
-Text Label 7200 5850 0    60   ~ 0
+Text Label 7200 3950 0    60   ~ 0
 LEVEL16_OK
 Text Label 11650 3350 2    60   ~ 0
@@
 Text Label 12850 3250 0    60   ~ 0
 LEVEL3_SENSE
-Text Label 8350 5950 0    60   ~ 0
+Text Label 8350 10100 0    60   ~ 0
 LEVEL1_TEST
-Text Label 7200 6050 0    60   ~ 0
+Text Label 7200 10200 0    60   ~ 0
 LEVEL3_TEST
 Text Label 7200 2550 0    60   ~ 0
@@
 L R R31
 U 1 1 5927C348
-P 7950 5950
-F 0 "R31" V 7900 6150 50  0000 C CNN
-F 1 "270" V 7950 5950 50  0000 C CNN
-F 2 "azonenberg_pcb:EIA_0402_RES_NOSILK" V 7880 5950 50  0001 C CNN
-F 3 "" H 7950 5950 50  0000 C CNN
-	1    7950 5950
+P 7950 10100
+F 0 "R31" V 7900 10300 50  0000 C CNN
+F 1 "270" V 7950 10100 50  0000 C CNN
+F 2 "azonenberg_pcb:EIA_0402_RES_NOSILK" V 7880 10100 50  0001 C CNN
+F 3 "" H 7950 10100 50  0000 C CNN
+	1    7950 10100
 	0    1    1    0
 $EndComp
@@
 L R R30
 U 1 1 5927CED4
-P 7950 6150
-F 0 "R30" V 7900 6350 50  0000 C CNN
-F 1 "0" V 7950 6150 50  0000 C CNN
-F 2 "azonenberg_pcb:EIA_0805_CAP_NOSILK" V 7880 6150 50  0001 C CNN
-F 3 "" H 7950 6150 50  0000 C CNN
-	1    7950 6150
+P 7950 11500
+F 0 "R30" V 7900 11700 50  0000 C CNN
+F 1 "0" V 7950 11500 50  0000 C CNN
+F 2 "azonenberg_pcb:EIA_0805_CAP_NOSILK" V 7880 11500 50  0001 C CNN
+F 3 "" H 7950 11500 50  0000 C CNN
+	1    7950 11500
 	0    1    1    0
 $EndComp
 Text Label 12850 3150 0    60   ~ 0
 LEVEL4_SENSE
-Text Label 8350 6150 0    60   ~ 0
+Text Label 8350 11500 0    60   ~ 0
 LEVEL4_TEST
 Text Label 7200 2750 0    60   ~ 0
 LEVEL4_SENSE
-Text Label 8350 6250 0    60   ~ 0
+Text Label 8350 11600 0    60   ~ 0
 LEVEL5_TEST
-Text Label 8350 6350 0    60   ~ 0
+Text Label 8350 9700 0    60   ~ 0
 LEVEL6_TEST
 Text Label 11650 2950 2    60   ~ 0
@@
 L R R38
 U 1 1 59282204
-P 7950 6250
-F 0 "R38" V 7900 6450 50  0000 C CNN
-F 1 "270" V 7950 6250 50  0000 C CNN
-F 2 "azonenberg_pcb:EIA_0402_RES_NOSILK" V 7880 6250 50  0001 C CNN
-F 3 "" H 7950 6250 50  0000 C CNN
-	1    7950 6250
+P 7950 11600
+F 0 "R38" V 7900 11800 50  0000 C CNN
+F 1 "270" V 7950 11600 50  0000 C CNN
+F 2 "azonenberg_pcb:EIA_0402_RES_NOSILK" V 7880 11600 50  0001 C CNN
+F 3 "" H 7950 11600 50  0000 C CNN
+	1    7950 11600
 	0    1    1    0
 $EndComp
@@
 L R R39
 U 1 1 592822E4
-P 7950 6350
-F 0 "R39" V 7900 6550 50  0000 C CNN
-F 1 "270" V 7950 6350 50  0000 C CNN
-F 2 "azonenberg_pcb:EIA_0402_RES_NOSILK" V 7880 6350 50  0001 C CNN
-F 3 "" H 7950 6350 50  0000 C CNN
-	1    7950 6350
+P 7950 9700
+F 0 "R39" V 7900 9900 50  0000 C CNN
+F 1 "270" V 7950 9700 50  0000 C CNN
+F 2 "azonenberg_pcb:EIA_0402_RES_NOSILK" V 7880 9700 50  0001 C CNN
+F 3 "" H 7950 9700 50  0000 C CNN
+	1    7950 9700
 	0    1    1    0
 $EndComp
@@
 Text Label 12850 4150 0    60   ~ 0
 LEVEL8_SENSE
-Text Label 7200 6450 0    60   ~ 0
+Text Label 7200 5750 0    60   ~ 0
 LEVEL8_TEST
 Text Label 7200 3050 0    60   ~ 0
@@
 L R R40
 U 1 1 59288963
-P 7950 6550
-F 0 "R40" V 7900 6750 50  0000 C CNN
-F 1 "270" V 7950 6550 50  0000 C CNN
-F 2 "azonenberg_pcb:EIA_01005_RES_NOSILK" V 7880 6550 50  0001 C CNN
-F 3 "" H 7950 6550 50  0000 C CNN
-	1    7950 6550
-	0    1    1    0
-$EndComp
-Text Label 7200 6550 0    60   ~ 0
+P 7950 7150
+F 0 "R40" V 7900 7350 50  0000 C CNN
+F 1 "270" V 7950 7150 50  0000 C CNN
+F 2 "azonenberg_pcb:EIA_01005_RES_NOSILK" V 7880 7150 50  0001 C CNN
+F 3 "" H 7950 7150 50  0000 C CNN
+	1    7950 7150
+	0    1    1    0
+$EndComp
+Text Label 7200 7150 0    60   ~ 0
 LEVEL9_TEST
-Text Label 8350 6550 0    60   ~ 0
+Text Label 8350 7150 0    60   ~ 0
 LEVEL9_SENSE
 Text Label 7200 3350 0    60   ~ 0
@@
 Text Label 8400 10900 0    60   ~ 0
 GND
-Text Label 7200 6950 0    60   ~ 0
+Text Label 7200 4050 0    60   ~ 0
 LEVEL17_OK
-Text Label 7200 7050 0    60   ~ 0
+Text Label 7200 3850 0    60   ~ 0
 LEVEL18_OK
 $Comp
@@
 	7000 5750 7200 5750
 Wire Wire Line
-	7200 5650 7000 5650
-Wire Wire Line
 	7000 3550 7200 3550
 Wire Wire Line
 	7200 3650 7000 3650
 Wire Wire Line
-	7000 3750 7200 3750
-Wire Wire Line
 	7200 3850 7000 3850
 Wire Wire Line
-	7000 3950 7200 3950
-Wire Wire Line
-	7200 4050 7000 4050
+	7000 9700 7800 9700
 Wire Wire Line
 	7000 4150 7200 4150
@@
 	7200 4250 7000 4250
 Wire Wire Line
-	7200 5150 7000 5150
-Wire Wire Line
 	7000 5250 7200 5250
 Wire Wire Line
@@
 	12850 3250 12750 3250
 Wire Wire Line
-	7200 6050 7000 6050
-Wire Wire Line
-	7000 5950 7800 5950
+	7200 10200 7000 10200
+Wire Wire Line
+	7000 10100 7800 10100
 Wire Wire Line
 	7200 2650 7000 2650
@@
 	7200 2750 7000 2750
 Wire Wire Line
-	7000 6150 7800 6150
-Wire Wire Line
-	7000 6350 7800 6350
-Wire Wire Line
-	7000 6250 7800 6250
-Wire Wire Line
-	8350 5950 8100 5950
-Wire Wire Line
-	8350 6150 8100 6150
-Wire Wire Line
-	8350 6250 8100 6250
-Wire Wire Line
-	8100 6350 8350 6350
+	7000 11500 7800 11500
+Wire Wire Line
+	7000 11600 7800 11600
+Wire Wire Line
+	8350 10100 8100 10100
+Wire Wire Line
+	8350 11500 8100 11500
+Wire Wire Line
+	8350 11600 8100 11600
+Wire Wire Line
+	8100 9700 8350 9700
 Wire Wire Line
 	11650 3250 11800 3250
@@
 	7200 3050 7000 3050
 Wire Wire Line
-	7000 6550 7800 6550
-Wire Wire Line
-	8350 6550 8100 6550
+	7000 7150 7800 7150
+Wire Wire Line
+	8350 7150 8100 7150
 Wire Wire Line
 	7200 3350 7000 3350
@@
 Wire Wire Line
 	800  9600 800  9500
-Text Label 7200 7150 0    60   ~ 0
+Text Label 7200 3750 0    60   ~ 0
 LEVEL19_OK
-Text Label 7200 7250 0    60   ~ 0
+Text Label 7200 3650 0    60   ~ 0
 LEVEL20_OK
 Text Label 7200 7350 0    60   ~ 0
 LEVEL21_OK
-Text Label 7200 7450 0    60   ~ 0
+Text Label 7200 3550 0    60   ~ 0
 LEVEL22_OK
 Wire Wire Line
@@
 Wire Wire Line
 	7200 7250 7000 7250
-Wire Wire Line
-	7000 7150 7200 7150
 $Comp
 L LED D20
@@
 NoConn ~ 2700 11800
 NoConn ~ 2700 11900
-NoConn ~ 7000 10100
-NoConn ~ 7000 10200
-NoConn ~ 7000 9700
 NoConn ~ 7000 9500
 NoConn ~ 7000 9200
 NoConn ~ 7000 9000
-NoConn ~ 7000 11500
-NoConn ~ 7000 11600
 NoConn ~ 7000 11900
 NoConn ~ 2700 12600
@@
 Connection ~ 4200 15050
 $Comp
-L R R?
+L R R52
 U 1 1 592C256B
 P 8800 1350
-F 0 "R?" V 8750 1200 50  0000 C CNN
+F 0 "R52" V 8750 1200 50  0000 C CNN
 F 1 "1K" V 8800 1350 50  0000 C CNN
 F 2 "azonenberg_pcb:EIA_0402_RES_NOSILK" V 8730 1350 50  0001 C CNN
@@
 Wire Wire Line
 	8650 1200 8800 1200
+Wire Wire Line
+	7200 6350 7000 6350
+Wire Wire Line
+	7200 6550 7000 6550
+NoConn ~ 7000 4950
+NoConn ~ 7000 5050
+Wire Wire Line
+	7200 3950 7000 3950
+Wire Wire Line
+	7000 5150 7200 5150
+Wire Wire Line
+	7200 4050 7000 4050
+Wire Wire Line
+	7200 3750 7000 3750
+NoConn ~ 7000 5650
+NoConn ~ 7000 6250
+NoConn ~ 7000 6150
+NoConn ~ 7000 6050
+NoConn ~ 7000 5950
 $EndSCHEMATC
