File: pcb/reworkctf.sch (KiCad schematic (older format))
At the start: 134 parts, among them J1 XILINX_JTAG, J2 UX60SX-MB-5ST, U1 XC3S50A-4FTG256C, U2 W25Q80BV, U3 74HC04, U4 1 MHz, U5 ADP322ACPZ-145-R7, U6 74HC04

Commit message: Finished initial work on rework challenge board
Parts:
- removed R34: 270, azonenberg_pcb:EIA_0402_RES_NOSILK, symbol R
- R41, R42: value 0 -> 270
Connections:
- net LEVEL11_SENSE: now also U1.E4 (IP_L04P_3); no longer U1.E3 (IO_L05P_3_NC_IN_50A)
- net LEVEL11_TEST: now also U1.E3 (IO_L05P_3_NC_IN_50A); no longer U1.E2 (IO_L05N_3_NC_IN_50A)
- net LEVEL12_SENSE: now also U1.R15 (IO_L02P_1/LDC1); no longer U1.L7 (IP_2)
- net LEVEL12_TEST: now also U1.P16 (IO_L03P_1/A0); no longer U1.T13 (IO_L18P_2/D2)
- net LEVEL13_TEST_A: now also U1.B3 (IO_L19N_0); no longer U1.L9 (IP_2/VREF_2)
- net LEVEL13_TEST_B: now also U1.A3 (IO_L19P_0); no longer U1.L8 (IP_2)
- net LEVEL14_SENSE: now also U1.J7 (IP_L13N_3); no longer U1.L10 (IP_2/VREF_2)
- net LEVEL14_TEST: now also U1.T9 (IO_L12N_2/GCLK3); no longer U1.R11 (IO_L15N_2/DOUT)
- net LEVEL15_TEST_N: now also U1.A13 (IO_L04N_0), U1.A8 (IO_L12P_0/GCLK10); no longer U1.A11 (IO_L07N_0), U1.C10 (IO_L09P_0/GCLK4)
- net LEVEL15_TEST_P: now also U1.A14 (IO_L04P_0), U1.B8 (IO_L12N_0/GCLK11); no longer U1.C11 (IO_L07P_0), U1.D9 (IO_L09N_0/GCLK5)
- net LEVEL16_TEST_A: now also R32.1, U1.T13 (IO_L18P_2/D2); no longer R32.2, U1.P16 (IO_L03P_1/A0)
- net LEVEL16_TEST_B: now also R33.1, U1.P13 (IO_L19N_2_NC_IN_50A); no longer R33.2, U1.M14 (IO_L05N_1/VREF_1_NC_IN_50A)
- net LEVEL19_SENSE: now also U1.J14 (IO_L14P_1/RHCLK4); no longer R41.1, U1.P8 (IO_L10P_2/GCLK14), U1.T5 (IO_L06P_2/D7)
- net LEVEL19_TEST: now also U1.E13 (IO_L23P_1/A22), U1.H15 (IO_L15P_1/IRDY1/RHCLK6); no longer U1.T6 (IO_L06N_2/D6), U1.T8 (IO_L10N_2/GCLK15)
- net LEVEL1_SENSE: now also U1.K15 (IO_L11P_1/RHCLK0); no longer U1.L5 (IP_L25P_3)
- net LEVEL20_OK: now also U1.J3 (IO_L12N_3/IRDY2/LHCLK3); no longer U1.M4 (IO_L24N_3)
- net LEVEL21_OK: now also U1.M4 (IO_L24N_3); no longer U1.C2 (IO_L01P_3)
- net LEVEL21_SENSE: now also U1.L5 (IP_L25P_3); no longer U1.K15 (IO_L11P_1/RHCLK0)
- net LEVEL21_TEST: now also R35.1; no longer R35.2
- net LEVEL22_SENSE: now also U1.E14 (IO_L20P_1/A18); no longer U1.K16 (IO_L12P_1/RHCLK2)
- net LEVEL22_TEST: now also U1.F13 (IO_L20N_1/A19); no longer U1.J16 (IO_L12N_1/TRDY1/RHCLK3)
- net LEVEL3_SENSE: now also U1.D15 (IO_L22N_1/A21); no longer U1.L6 (IP_L25N_3/VREF_3)
- net LEVEL3_TEST: now also U1.D16 (IO_L22P_1/A20); no longer U1.T9 (IO_L12N_2/GCLK3)
- net LEVEL4_SENSE: now also U1.C15 (IO_L24N_1/A25); no longer U1.K5 (IP_L21P_3)
- net LEVEL4_TEST: now also R30.2; no longer R30.1
- net LEVEL5_SENSE: now also U1.H14 (IO_L14N_1/RHCLK5); no longer U1.K6 (IP_L21N_3)
- net LEVEL6_SENSE: now also U1.D14 (IO_L23N_1/A23); no longer U1.H7 (IP_L13P_3)
- net LEVEL7_TEST_N: now also U1.A12 (IO_L05N_0_NC_IN_50A); no longer U1.C13 (IO_L01N_0)
- net LEVEL7_TEST_P: now also U1.B12 (IO_L05P_0); no longer U1.D13 (IO_L01P_0)
- net LEVEL8_SENSE: now also U1.H7 (IP_L13P_3); no longer U1.J7 (IP_L13N_3)
- net LEVEL9_SENSE: now also R40.2, U1.A5 (IO_L17P_0); no longer R40.1, U1.E4 (IP_L04P_3)
- net LEVEL9_TEST: now also R40.1, U1.A4 (IO_L18P_0); no longer R40.2, U1.D4 (IO_L02P_3)
- net at U1.C16 (IO_L24P_1/A24): now also R30.1
- net at U1.C8 (IO_L11P_0/GCLK8): now also R36.2
- net at U1.D7 (IO_L16P_0): now also R37.2
- net at U1.H16 (IO_L15N_1/RHCLK7): now also R41.1
- net at U1.K14 (IO_L11N_1/RHCLK1): now also R39.2; no longer R35.1
- net at U1.N11 (IO_L16N_2): no longer R37.2
- net at U1.N13 (IO_L01P_1/HDC): no longer R32.1
- net at U1.N16 (IO_L03N_1/A1): now also R31.2
- net at U1.P11 (IO_L16P_2): no longer R36.2
- net at U1.P15 (IO_L02N_1/LDC0): no longer R33.1
- net at R38.2: now also U1.K16 (IO_L12P_1/RHCLK2); no longer U1.R5 (IO_L05N_2)
- net at U1.R9 (IO_L12P_2/GCLK2): no longer R31.2
- net at U1.T10 (IO_L14P_2): no longer R39.2
- net at U1.T4 (IO_L05P_2): now also R32.2; no longer R30.2
- net LEVEL16_TEST_C: no longer names the net of U1.M13 (IO_L05P_1_NC_IN_50A)
- new net: R33.2, U1.R11 (IO_L15N_2/DOUT)
- new net: R35.2, U1.T8 (IO_L10N_2/GCLK15)
- no-connect marks 121 -> 123
Other:
- note added: "IO_L12 pair\nintentionally swapped"
- note removed: "IO_L09 pair\nintentionally swapped"
- moved on the sheet: R30, R31, R32, R33, R35, R36, R37, R38, R39, R40, R41, R42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
