File: v2/pcb/reworkctf-v2.kicad_pcb (KiCad board)
At the start: 4 copper layers, 54 x 50 mm, 106 parts, among them J1 USB_C_Receptacle_USB2.0, J2 CORTEX_DEBUG_ETM, J3 DOT, J4 TESTPOINT, J6 CONN_01X03, J7 PMOD_HOST, J8 PMOD_HOST, M1 SCREWHOLE, M2 SCREWHOLE, M3 SCREWHOLE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

Commit message: Initial work on "free play area" sandbox
Parts:
- added R39: R, azonenberg_pcb:EIA_0402_RES_NOSILK, F.Cu at (66.2, 56.8)
- added R40: R, azonenberg_pcb:EIA_0402_RES_NOSILK, F.Cu at (66.2, 57.5)
- added R41: R, azonenberg_pcb:EIA_0402_RES_NOSILK, F.Cu at (66.2, 58.2)
- added R42: R, azonenberg_pcb:EIA_0402_RES_NOSILK, F.Cu at (66.2, 59.0)
- added R43: R, azonenberg_pcb:EIA_0402_RES_NOSILK, F.Cu at (66.2, 59.8)
- added R44: R, azonenberg_pcb:EIA_0402_RES_NOSILK, F.Cu at (66.2, 60.5)
- added R45: R, azonenberg_pcb:EIA_0402_RES_NOSILK, F.Cu at (66.2, 61.2)
- added R46: R, azonenberg_pcb:EIA_0402_RES_NOSILK, F.Cu at (66.2, 62.0)
- added R47: R, azonenberg_pcb:EIA_0402_RES_NOSILK, F.Cu at (68.8, 56.8)
- added R48: R, azonenberg_pcb:EIA_0402_RES_NOSILK, F.Cu at (68.8, 57.5)
- added R49: R, azonenberg_pcb:EIA_0402_RES_NOSILK, F.Cu at (68.8, 58.2)
- added R50: R, azonenberg_pcb:EIA_0402_RES_NOSILK, F.Cu at (68.8, 59.0)
- added R51: R, azonenberg_pcb:EIA_0402_RES_NOSILK, F.Cu at (68.8, 59.8)
- added R52: R, azonenberg_pcb:EIA_0402_RES_NOSILK, F.Cu at (68.8, 60.5)
- added R53: R, azonenberg_pcb:EIA_0402_RES_NOSILK, F.Cu at (68.8, 61.2)
Routing:
- net (no net): track 0.00 -> 133.0 mm
- net unconnected-(R52-Pad2): track 0.00 -> 6.50 mm, vias 0 -> 1
- net unconnected-(R50-Pad2): track 0.00 -> 6.50 mm, vias 0 -> 1
- net unconnected-(R48-Pad2): track 0.00 -> 6.50 mm, vias 0 -> 1
- net unconnected-(R53-Pad2): track 0.00 -> 6.00 mm, vias 0 -> 1
- net unconnected-(R51-Pad2): track 0.00 -> 6.00 mm, vias 0 -> 1
- net unconnected-(R49-Pad2): track 0.00 -> 6.00 mm, vias 0 -> 1
- net unconnected-(R47-Pad2): track 0.00 -> 6.00 mm, vias 0 -> 1
- net unconnected-(R46-Pad1): track 0.00 -> 1.25 mm
- net unconnected-(R45-Pad1): track 0.00 -> 1.25 mm
- net unconnected-(R44-Pad1): track 0.00 -> 1.25 mm
- net unconnected-(R43-Pad1): track 0.00 -> 1.25 mm
- net unconnected-(R42-Pad1): track 0.00 -> 1.25 mm
- net unconnected-(R41-Pad1): track 0.00 -> 1.25 mm
- net unconnected-(R40-Pad1): track 0.00 -> 1.25 mm
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Other:
- board text added: "<CH15"
- board text added: "Free Play Area"

Commit message: Added more inner layer test features to free play area
Parts:
- added J10: TESTPOINT, azonenberg_pcb:TESTPOINT_SMT_0.5MM, F.Cu at (72.0, 65.5)
- added J11: TESTPOINT, azonenberg_pcb:TESTPOINT_SMT_0.5MM, F.Cu at (76.0, 65.5)
- added J12: TESTPOINT, azonenberg_pcb:TESTPOINT_SMT_0.5MM, F.Cu at (73.8, 63.0)
- added J13: TESTPOINT, azonenberg_pcb:TESTPOINT_SMT_0.5MM, F.Cu at (74.5, 63.0)
- added J14: TESTPOINT, azonenberg_pcb:TESTPOINT_SMT_0.5MM, F.Cu at (73.8, 67.0)
- added J15: TESTPOINT, azonenberg_pcb:TESTPOINT_SMT_0.5MM, F.Cu at (74.5, 67.0)
- added J16: TESTPOINT, azonenberg_pcb:TESTPOINT_SMT_0.5MM, F.Cu at (76.0, 63.0)
- added J17: TESTPOINT, azonenberg_pcb:TESTPOINT_SMT_0.5MM, F.Cu at (72.0, 63.0)
- added J5: TESTPOINT, azonenberg_pcb:TESTPOINT_SMT_0.5MM, F.Cu at (72.0, 64.8)
- added J9: TESTPOINT, azonenberg_pcb:TESTPOINT_SMT_0.5MM, F.Cu at (76.0, 64.8)
Routing:
- net /GND: track 338.5 -> 352.9 mm, vias 83 -> 84
- net /3V3: track 201.5 -> 213.1 mm, vias 36 -> 37
- net Net-(J5-P1): track 0.00 -> 4.21 mm
- net Net-(J13-P1): track 0.00 -> 4.21 mm, vias 0 -> 2
- net Net-(J12-P1): track 0.00 -> 4.21 mm, vias 0 -> 2
- net Net-(J10-P1): track 0.00 -> 4.21 mm
